File: TestBoard/MCU/MCU.kicad_sch (KiCad schematic)
At the start: 3 parts, among them J1 Rail Left, J2 Rail Right, U1 STM32G431CBTx

Commit message: MCU Done
Parts:
- added C1, C2: C, Capacitor_SMD:C_0603_1608Metric_Pad1.08x0.95mm_HandSolder, symbol Device:C
Connections:
- net 19 is gone; now on net GND: J1.19 (Pin_19), U1.19 (VSSA)
- net 21 is gone; now on net VDD: J1.21 (Pin_21), U1.21 (VDDA)
- net 23 is gone; now on net GND: J1.23 (Pin_23), U1.23 (VSS), U1.35 (VSS), U1.47 (VSS)
- net 24 is gone; now on net VDD: J1.24 (Pin_24), U1.24 (VDD)
- net 36 is gone; now on net VDD: J2.12 (Pin_12), U1.36 (VDD)
- net 48 is gone; now on net VDD: J2.24 (Pin_24), U1.48 (VDD)
- net VDD: now reaches J1.1 (Pin_1), U1.1 (VBAT)
- net VDD: now also C1.1, C2.1
- net GND: now reaches J2.11 (Pin_11)
- net GND: now also J2.23 (Pin_23), C1.2, C2.2
- no-connect marks 2 -> 0
