File: TestBoard/MagEncoder/MagEncoder/MagEncoder.kicad_pcb (KiCad board)
At the start: 2 copper layers, 23.4 x 23.3 mm, 8 parts, among them J1 Conn_01x05_Pin, U1 MT6701QT

Commit message: Mag Encoder Done
Parts:
- removed TP1: TestPoint, TestPoint:TestPoint_Pad_1.0x1.0mm
- added J2: Conn_01x05_Pin, Connector_JST:JST_GH_SM05B-GHS-TB_1x05-1MP_P1.25mm_Horizontal, B.Cu at (153.2, 102.8)
- C1: footprint Capacitor_SMD:C_0402_1005Metric -> Capacitor_SMD:C_0805_2012Metric_Pad1.18x1.45mm_HandSolder; moved to B.Cu
- JP1: footprint Jumper:SolderJumper-2_P1.3mm_Open_TrianglePad1.0x1.5mm -> Jumper:SolderJumper-2_P1.3mm_Bridged_RoundedPad1.0x1.5mm
- R1, R2: footprint Resistor_SMD:R_0402_1005Metric -> Resistor_SMD:R_0603_1608Metric_Pad0.98x0.95mm_HandSolder; moved to B.Cu
- REF**: moved to B.Cu
- moved R1 8.02 mm to (142.8, 101.2), turned to 45 degrees
- moved R2 4.44 mm to (141.2, 99.8), turned to 45 degrees
- moved C1 1.96 mm to (147.0, 95.3), turned to -90 degrees
- turned REF** to 180 degrees
Connections:
- J1 pad MP: GND -> (no net)
- U1 pad 11: unconnected-(U1-U-Pad11) -> Net-(J2-Pin_3)
- U1 pad 12: unconnected-(U1-V-Pad12) -> Net-(J2-Pin_2)
- U1 pad 9: unconnected-(U1-W-Pad9) -> Net-(J2-Pin_4)
Routing:
- net GND: track 1.25 -> 28.6 mm, vias 7 -> 6
- net Net-(J2-Pin_1): track 6.74 -> 17.3 mm
- net Net-(J2-Pin_2): track 0.00 -> 8.67 mm, vias 0 -> 1
- net Net-(J2-Pin_3): track 0.00 -> 8.32 mm, vias 0 -> 1
- net Net-(J2-Pin_4): track 0.00 -> 7.15 mm, vias 0 -> 1
- net +5V: track 20.8 -> 18.3 mm, vias 2 -> 5
- net /SCL/CLK: track 17.0 -> 15.1 mm
- net /VDD/CSN: track 20.1 -> 21.9 mm, vias 1 -> 3
- net /SDA/DO: track 16.8 -> 15.3 mm
- net (no net): vias 1 -> 0
- added copper zone on F.Cu, net +5V
- removed copper zone on F.Cu, net GND
Other:
- board text added: "+"
- board text added: "G"
- board text added: "PUSH"
- board text added: "SCL"
- board text added: "SDA"
- board text added: "U"
- board text added: "V"
- board text added: "W"
