File: FinalBoard/FinalBoard.kicad_sch (KiCad schematic)
At the start: 42 parts, among them J1 Power Input, J2 NRF24L01P, J3 Motor Output, J4 Position_Sensor, J5 Programming, J6 UART, J7 Conn_01x28, U1 DRV8316RRGFR, U4 LT1086-3.3, U5 STM32G431VBTx

Commit message: Position sensor worky
Parts:
- C3: value 100n -> 100nF
- C5: value 47n -> 47nF
- R10, R12, R8: value R -> 10k
- R11, R2, R7, R9: value R -> 3.9k
- R3, R4, R5, R6: value R -> 470
Changed lines of the file:
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@@
 			)
 		)
-		(property "Value" "R"
+		(property "Value" "470"
 			(at 52.07 74.9299 0)
 			(effects
@@
 			)
 		)
-		(property "Value" "47n"
+		(property "Value" "47nF"
 			(at 176.53 63.4999 0)
 			(effects
@@
 			)
 		)
-		(property "Value" "R"
+		(property "Value" "3.9k"
 			(at 240.03 44.45 90)
 			(effects
@@
 			)
 		)
-		(property "Value" "100n"
+		(property "Value" "100nF"
 			(at 166.37 76.1999 0)
 			(effects
@@
 			)
 		)
-		(property "Value" "R"
+		(property "Value" "10k"
 			(at 254 54.61 90)
 			(effects
@@
 			)
 		)
-		(property "Value" "R"
+		(property "Value" "3.9k"
 			(at 240.03 54.61 90)
 			(effects
@@
 			)
 		)
-		(property "Value" "R"
+		(property "Value" "470"
 			(at 64.77 74.9299 0)
 			(effects
@@
 			)
 		)
-		(property "Value" "R"
+		(property "Value" "470"
 			(at 39.37 74.9299 0)
 			(effects
@@
 			)
 		)
-		(property "Value" "R"
+		(property "Value" "10k"
 			(at 254 64.77 90)
 			(effects
@@
 			)
 		)
-		(property "Value" "R"
+		(property "Value" "10k"
 			(at 254 44.45 90)
 			(effects
@@
 			)
 		)
-		(property "Value" "R"
+		(property "Value" "3.9k"
 			(at 149.86 113.0299 0)
 			(effects
@@
 			)
 		)
-		(property "Value" "R"
+		(property "Value" "470"
 			(at 22.86 74.9299 0)
 			(effects
@@
 			)
 		)
-		(property "Value" "R"
+		(property "Value" "3.9k"
 			(at 240.03 64.77 90)
 			(effects
